File: uEFI_rev3/uEFI_rev3.kicad_sch (KiCad schematic)
At the start: 89 parts, among them J1 USB_B, J2 Tag connect, J4 Conn_02x08_Odd_Even, J5 Conn_01x03, Q11 SS8050, Q12 AO3400A, Q13 AO3400A, Q8 SS8050, Q9 SS8050, SW1 SW_Push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

Commit message: Update uEFI_rev3.kicad_sch
Other:
- title: uEFI -> uEF I
Changed lines of the file:
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@@
   (paper "A3")
   (title_block
-    (title "uEFI")
+    (title "uEF I")
     (date "%%date%%")
     (rev "v3-%%version%%")
